File: PCB/Recept/Recept.kicad_sch (KiCad schematic)
At the start: 0 parts

Commit message: Update
Parts:
- added C1, C10, C103, C104, C105, C110, C111, C113, C115, C117, C119, C12, C4, C5, C6, C7, C8: 0.1uF, Capacitor_SMD:C_0402_1005Metric, symbol Device:C
- added C100: 33uF, Capacitor_SMD:C_0603_1608Metric, symbol Device:C
- added C101, C85, C87, C92, C94, C97: 10uF, Capacitor_SMD:C_0603_1608Metric, symbol Device:C
- added C102: 1uF, Capacitor_SMD:C_0603_1608Metric, symbol Device:C
- added C106, C95: 20pF, Capacitor_SMD:C_0402_1005Metric, symbol Device:C
- added C107: 220nF, Capacitor_SMD:C_0402_1005Metric, symbol Device:C
- added C108, C109, C11, C112, C114, C116, C118, C81, C82: 10uF, Capacitor_SMD:C_0402_1005Metric, symbol Device:C
- added C2, C9: 10pF, Capacitor_SMD:C_0402_1005Metric, symbol Device:C
- added C3, C96: 1uF, Capacitor_SMD:C_0402_1005Metric, symbol Device:C
- added C83, C84: 10uF, Capacitor_SMD:C_0805_2012Metric, symbol Device:C
- added C86: 100nF, Capacitor_SMD:C_0402_1005Metric, symbol Device:C
- added C88, C89, C90: 22uF, Capacitor_SMD:C_0805_2012Metric, symbol Device:C
- added C91, C93: 100nF, Capacitor_SMD:C_0603_1608Metric, symbol Device:C
- added C98: 22uF, Capacitor_SMD:C_0603_1608Metric, symbol Device:C
- added C99: 4.7uF, Capacitor_SMD:C_0603_1608Metric, symbol Device:C
- added CM1: RX5808, lcsc:COMM-SMD_12P_RX5808, symbol LCSC:RX5808
- added D10: Diode, Diode_SMD:D_SMB, symbol Device:D
- added FPC1: 0.5K-AS-40PWB, lcsc:FPC-SMD_40P-P0.50_0.5K-AS-40PWB, symbol LCSC:0.5K-AS-40PWB
- added J1: Conn_01x02_Pin, Connector_PinHeader_2.54mm:PinHeader_1x02_P2.54mm_Vertical, symbol Connector:Conn_01x02_Pin
- added J2: Conn_02x03_Counter_Clockwise, Connector_PinHeader_1.27mm:PinHeader_2x03_P1.27mm_Vertical, symbol Connector_Generic:Conn_02x03_Counter_Clockwise
- added J4: Conn_02x04_Counter_Clockwise, Connector_PinHeader_1.27mm:PinHeader_2x04_P1.27mm_Vertical, symbol Connector_Generic:Conn_02x04_Counter_Clockwise
- added J5: Conn_02x02_Counter_Clockwise, Connector_PinHeader_1.27mm:PinHeader_2x02_P1.27mm_Vertical, symbol Connector_Generic:Conn_02x02_Counter_Clockwise
- added L3: XFL4020-152MEC, LCSC:IND-SMD_L4.0-W4.0-A, symbol LCSC:XFL4020-152MEC
- added L4: 22uH, LCSC:IND-SMD_L5.8-W5.8, symbol Device:L_Ferrite
- added LED1, LED2, LED3, LED4, LED5, LED6, LED7, LED8: KT-0603YB, LCSC:LED0603-RD, symbol LCSC:XL-0603QYGC
- added LED10, LED17, LED18, LED19, LED20, LED21, LED22: KT-0603YG, LCSC:LED0603-RD, symbol LCSC:XL-0603QYGC
- added LED23: KT-0603YR, LCSC:LED0603-RD, symbol LCSC:XL-0603QYGC
- added R1, R116, R2, R3, R4, R5, R6, R7, R8, R90: 220, Resistor_SMD:R_0402_1005Metric, symbol Device:R
- added R10, R9: 27, Resistor_SMD:R_0402_1005Metric, symbol Device:R
- added R105: 396K, Resistor_SMD:R_0402_1005Metric, symbol Device:R
- added R106, R12, R70, R81, R91, R92, R95: 10K, Resistor_SMD:R_0402_1005Metric, symbol Device:R
- added R107, R13, R14, R15, R16: 4.7K, Resistor_SMD:R_0402_1005Metric, symbol Device:R
- added R108: 2.2K, Resistor_SMD:R_0402_1005Metric, symbol Device:R
- added R11, R94: 1K, Resistor_SMD:R_0402_1005Metric, symbol Device:R
- added R111, R112, R113: 1.5K, Resistor_SMD:R_0402_1005Metric, symbol Device:R
- added R114: 3.3K, Resistor_SMD:R_0402_1005Metric, symbol Device:R
- added R115: 1.5k, Resistor_SMD:R_0402_1005Metric, symbol Device:R
- added R57, R59: 5.1K, Resistor_SMD:R_0402_1005Metric, symbol Device:R
- added R71: 100K, Resistor_SMD:R_0402_1005Metric, symbol Device:R
- added R79: 80, Resistor_SMD:R_0402_1005Metric, symbol Device:R
- added R93: 1.8K, Resistor_SMD:R_0402_1005Metric, symbol Device:R
- added RV1: 10K, Potentiometer_SMD:Potentiometer_Bourns_3314J_Vertical, symbol Device:R_Potentiometer
- added SW1, SW16: SW_Push, Button_Switch_SMD:SW_Push_1P1T-SH_NO_CK_KMR2xxG, symbol Switch:SW_Push
- added SW15: DSIC03LSGET, LCSC:SW-SMD_DSIC03LSGET, symbol LCSC:DSIC03LSGET
- added SW18: K3-1204D-L, lcsc:SW-TH_K3-1204D-L, symbol LCSC:K3-1204D-L
- added U1: RP2040, Package_DFN_QFN:QFN-56-1EP_7x7mm_P0.4mm_EP3.2x3.2mm, symbol MCU_RaspberryPi:RP2040
- added U2: ABM8-272-T3_C20625731, lcsc:CRYSTAL-SMD_4P-L3.2-W2.5-BL, symbol LCSC:ABM8-272-T3_C20625731
- added U22: ~, Package_DFN_QFN:QFN-48-1EP_7x7mm_P0.5mm_EP5.6x5.6mm_ThermalVias, symbol my:TW8819
- added U24: TPS630701RNMT, LCSC:VQFN-15_L3.0-W2.5-P0.50-BL, symbol LCSC:TPS630701RNMT
- added U25: BQ21088YBGR, lcsc:DSBGA-8_L1.5-W1.0-R2-C4-P0.40-BL, symbol LCSC:BQ21088YBGR
- added U27: LD1117S33TR_SOT223, Package_TO_SOT_SMD:SOT-223-3_TabPin2, symbol Regulator_Linear:LD1117S33TR_SOT223
- added U28: CAT4104, LCSC:SOIC-8_L4.9-W3.9-P1.27-LS6.0-BL, symbol My_Library:CAT4104
- added U29: MT3608, Package_TO_SOT_SMD:SOT-23-6, symbol Regulator_Switching:MT3608
- added U30: SMA_Conn, LCSC:SMA-TH_SMA-KWE_C7498154, symbol LCSC:SMA-KWE_C7498154
- added U31: LD1117S18TR_SOT223, Package_TO_SOT_SMD:SOT-223-3_TabPin2, symbol Regulator_Linear:LD1117S18TR_SOT223
- added U4: W25Q16JVZPIQ, lcsc:WSON-8_L6.0-W5.0-P1.27-BL-EP, symbol LCSC:W25Q16JVZPIQ
- added USB2: TYPE-C 16P(073), LCSC:USB-C-SMD_TYPE-C16PIN_C668624, symbol LCSC:TYPE-C16P(073)
- added X3: X322527MSB4SI, lcsc:CRYSTAL-SMD_4P-L3.2-W2.5-BL-1, symbol LCSC:X322527MSB4SI
Connections:
- new net: LED17.2 (A), R112.2
- new net: LED19.2 (A), R114.2
- new net: R93.1, RV1.3
- new net: LED23.2 (A), R90.2
- new net: LED5.2 (A), R5.2
- new net: CM1.9 (RSSI), R108.1
- new net: LED3.2 (A), R3.2
- new net: R10.2, U1.46 (USB_DM)
- new net: R9.2, U1.47 (USB_DP)
- new net: D10.2 (A), L4.2, U29.1 (SW)
- new net: LED6.2 (A), R6.2
- new net: C100.1, SW18.3, U25.B2 (SYS)
- new net: LED21.2 (A), R116.2
- new net: CM1.2 (ANT), U30.5
- new net: CM1.4 (CH1), SW15.6 (B1)
- new net: CM1.5 (CH2), SW15.5 (B2)
- new net: CM1.6 (CH3), SW15.4 (B3)
- new net: R105.2, R95.1, U29.3 (FB)
- new net: R57.1, USB2.A5 (CC1)
- new net: LED10.2 (A), R111.2
- new net: C86.1, U24.3 (VAUX)
- new net: LED2.2 (A), R2.2
- new net: LED1.2 (A), R1.2
- new net: L3.1, U24.11 (L1)
- new net: L3.2, U24.9 (L2)
- new net: LED18.2 (A), R113.2
- new net: LED7.2 (A), R7.2
- new net: LED8.2 (A), R8.2
- new net: R70.2, U24.1 (PS/S), U24.14 (EN)
- new net: R71.1, U24.2 (PG)
- new net: R11.1, SW1.2
- new net: R106.1, U25.D1 (TS/MR)
- new net: LED4.2 (A), R4.2
- new net: R79.2, U22.10 (XTI)
- new net: C107.2, U22.2 (DIAG0/YIN0+/YIN1)
- new net: LED20.2 (A), R115.2
- new net: R93.2, U28.8 (RSET)
- new net: R59.1, USB2.B5 (CC2)
- new net: R94.1, U28.6 (EN/PWM)
- new net +1.1V: C3.1, C8.1, U1.23 (DVDD), U1.45 (VREG_VOUT), U1.50 (DVDD)
- new net +1.8V: C108.1, C11.2, C111.1, C112.2, C113.2, C116.2, C117.2, C12.2, C94.2, J4.4 (Pin_4), LED22.2 (A), U22.1 (AVDAD), U22.22 (VDD18), U22.42 (VDD18), U22.47 (AVDPLL), U31.2 (VO)
- new net +24V: C98.2, D10.1 (K), FPC1.2, J4.1 (Pin_1), R105.1, R114.1
- new net +3.3V: C1.1, C10.2, C102.1, C103.1, C104.1, C105.1, C109.2, C110.2, C114.1, C115.1, C4.1, C5.1, C6.1, C7.1, C92.2, FPC1.4, J4.3 (Pin_3), J5.1 (Pin_1), R116.1, R12.2, R13.1, R14.1, R15.1, R81.2, U1.1 (IOVDD), U1.10 (IOVDD), U1.22 (IOVDD), U1.33 (IOVDD), U1.42 (IOVDD), U1.43 (ADC_AVDD), U1.44 (VREG_IN), U1.48 (USB_VDD), U1.49 (IOVDD), U22.18 (VDD33), U22.37 (VDD33), U27.2 (VO), U4.8 (VCC)
- new net +5V: C118.1, C119.1, C87.2, C88.2, C89.2, C90.2, C91.2, CM1.8 (+5V), J4.2 (Pin_2), R115.1, R71.2, R94.2, U24.5 (FB), U24.7 (VOUT), U27.3 (VI), U28.7 (VIN)
- new net B0: FPC1.21, U22.17 (PWM1/TRSPB/FPB0)
- new net B1: FPC1.22, U22.19 (PWM2/CSPR/FPB1)
- new net B2: FPC1.23, U22.40 (FPB2)
- new net B3: FPC1.24, U22.41 (FPB3)
- new net B4: FPC1.25, U22.43 (FPB4)
- new net B5: FPC1.26, U22.44 (FPB5)
- new net B6: FPC1.27, U22.45 (FPB6)
- new net B7: FPC1.28, U22.46 (FPB7)
- new net BQ_INT: U1.16 (GPIO13), U25.A1 (~{INT})
- new net DE: FPC1.34, U22.16 (TROE/sDE/FPDE)
- new net DISP: FPC1.31, R15.2, U1.4 (GPIO2)
- new net DIVIDER: R91.2, R92.1, U1.39 (GPIO27_ADC1)
- new net G0: FPC1.13, U22.20 (GPIO1/TCLP/FPG0)
- new net G1: FPC1.14, U22.21 (GPIO2/TRUD/FPG1)
- new net G2: FPC1.15, U22.32 (FPG2/sD1)
- new net G3: FPC1.16, U22.33 (FPG3/sD0)
- new net G4: FPC1.17, U22.34 (FPG4)
- new net G5: FPC1.18, U22.35 (FPG5)
- new net G6: FPC1.19, U22.38 (FPG6)
- new net G7: FPC1.20, U22.39 (FPG7)
- new net GND: C1.2, C10.1, C100.2, C101.2, C102.2, C103.2, C104.2, C105.2, C106.2, C108.2, C109.1, C11.1, C110.1, C111.2, C112.1, C113.1, C114.2, C115.2, C116.1, C117.1, C118.2, C119.2, C12.1, C2.1, C3.2, C4.2, C5.2, C6.2, C7.2, C8.2, C81.2, C82.2, C83.1, C84.1, C85.1, C86.2, C87.1, C88.1, C89.1, C9.2, C90.1, C91.1, C92.1, C93.1, C94.1, C95.1, C96.1, C97.1, C98.1, C99.2, CM1.1 (GND), CM1.12 (GND), CM1.3 (GND), CM1.7 (GND), FPC1.29, FPC1.3, FPC1.36, FPC1.41, FPC1.42, J1.1 (Pin_1), J4.5 (Pin_5), J4.6 (Pin_6), J5.2 (Pin_2), LED1.1 (K), LED10.1 (K), LED17.1 (K), LED18.1 (K), LED19.1 (K), LED2.1 (K), LED20.1 (K), LED21.1 (K), LED22.1 (K), LED23.1 (K), LED3.1 (K), LED4.1 (K), LED5.1 (K), LED6.1 (K), LED7.1 (K), LED8.1 (K), R106.2, R107.2, R16.1, R57.2, R59.2, R91.1, R95.2, RV1.2, SW1.1, SW15.1 (A1), SW15.2 (A2), SW15.3 (A3), SW16.2, U1.19 (TESTEN), U1.57 (GND), U2.2 (GND), U2.4 (GND), U22.25 (VSS), U22.3 (DIAG1/YIN0-/YIN1), U22.36 (VSS), U22.4 (DIAG2/YIN2+/YIN2), U22.48 (AVSPLL), U22.5 (DIAG3/YIN2-/YIN3), U22.6 (AVSAD), U24.10 (PGND), U24.15 (VSEL), U24.4 (GND), U24.6 (FB2), U25.D2 (GND), U27.1 (GND), U28.5 (GND), U29.2 (GND), U30.1, U30.2, U30.3, U30.4, U31.1 (GND), U4.4 (GND), U4.9 (EP), USB2.1 (SHELL), USB2.2 (SHELL), USB2.3 (SHELL), USB2.4 (SHELL), USB2.A1B12 (GND), USB2.B1A12 (GND), X3.2 (GND), X3.4 (GND)
- new net GPIO14: J2.1 (Pin_1), U1.17 (GPIO14)
- new net GPIO15: J2.2 (Pin_2), U1.18 (GPIO15)
- new net GPIO16: J2.3 (Pin_3), U1.27 (GPIO16)
- new net GPIO17: J2.4 (Pin_4), U1.28 (GPIO17)
- new net GPIO18: J2.5 (Pin_5), U1.29 (GPIO18)
- new net GPIO19: J2.6 (Pin_6), U1.30 (GPIO19)
- new net GPIO_LED: R90.1, U1.37 (GPIO25)
- new net HSE_IN: C106.1, R79.1, X3.3 (OSC2)
- new net HSE_OUT: C95.2, U22.11 (XTO), X3.1 (OSC1)
- new net HSYNC: FPC1.32, U22.15 (TCSPL/sHS/FPHS)
- new net LED1: R1.1, U1.6 (GPIO4)
- new net LED2: R2.1, U1.7 (GPIO5)
- new net LED3: R3.1, U1.8 (GPIO6)
- new net LED4: R4.1, U1.9 (GPIO7)
- new net LED5: R5.1, U1.11 (GPIO8)
- new net LED6: R6.1, U1.12 (GPIO9)
- new net LED7: R7.1, U1.13 (GPIO10)
- new net LED8: R8.1, U1.14 (GPIO11)
- new net PCLK: FPC1.30, U22.13 (TCCLK/sCLK/FPCLK)
- new net QSPI_SCLK: U1.52 (QSPI_SCLK), U4.6 (CLK)
- new net QSPI_SD0: U1.53 (QSPI_SD0), U4.5 (DI(IO0))
- new net QSPI_SD1: U1.55 (QSPI_SD1), U4.2 (DO(IO1))
- new net QSPI_SD2: U1.54 (QSPI_SD2), U4.3 (WP#(IO2))
- new net QSPI_SD3: U1.51 (QSPI_SD3), U4.7 (~{HOLD}/RESET#(IO3))
- new net QSPI_SS: R11.2, R12.1, U1.56 (QSPI_SS), U4.1 (~{CS})
- new net R0: FPC1.5, U22.23 (GPIO3/TRCLK/FPR0)
- new net R1: FPC1.6, U22.24 (GPIO4/TCLRL/FPR1)
- new net R2: FPC1.7, U22.26 (FPR2/sD7)
- new net R3: FPC1.8, U22.27 (FPR3/sD6)
- new net R4: FPC1.9, U22.28 (FPR4/sD5)
- new net R5: FPC1.10, U22.29 (FPR5/sD4)
- new net R6: FPC1.11, U22.30 (FPR6/sD3)
- new net R7: FPC1.12, U22.31 (FPR7/sD2)
- new net RESET_TW8819: R16.2, U1.15 (GPIO12), U22.7 (RSTB)
- new net RSSI: R107.1, R108.2, U1.38 (GPIO26_ADC0)
- new net RUN: C96.2, R81.1, SW16.1, U1.26 (RUN)
- new net SCL: J4.7 (Pin_7), R14.2, U1.3 (GPIO1), U22.9 (SCL), U25.B1 (SCL)
- new net SDA: J4.8 (Pin_8), R13.2, U1.2 (GPIO0), U22.8 (SDA), U25.C1 (SDA)
- new net SWCLK: J5.4 (Pin_4), U1.24 (SWCLK)
- new net SWD: J5.3 (Pin_3), U1.25 (SWD)
- new net USB_DN: R10.1, USB2.A7 (DN1), USB2.B7 (DN2)
- new net USB_DP: R9.1, USB2.A6 (DP1), USB2.B6 (DP2)
- new net VBAT: C101.1, J1.2 (Pin_2), R112.1, R92.2, U25.C2 (BAT)
- new net VBUS: C81.1, C82.1, C99.1, R111.1, U25.A2 (IN), USB2.A4B9 (VBUS), USB2.B4A9 (VBUS)
- new net VIDEO: C107.1, CM1.11 (VIDEO)
- new net VLED-: FPC1.1, U28.1 (LED1)
- new net VSYNC: FPC1.33, U22.14 (TRSPT/sVS/FPVS)
- new net VSYS: C83.2, C84.2, C85.2, C93.2, C97.2, L4.1, R113.1, R70.1, SW18.2, U24.12 (VIN), U29.4 (EN), U29.5 (IN), U31.3 (VI)
- new net XIN: C9.1, U1.20 (XIN), U2.3
- new net XL: FPC1.39, U1.40 (GPIO28_ADC2)
- new net XOUT: C2.2, U1.21 (XOUT), U2.1
- new net XR: FPC1.37, U1.35 (GPIO23)
- new net YD: FPC1.38, U1.36 (GPIO24)
- new net YU: FPC1.40, U1.41 (GPIO29_ADC3)
- no-connect marks 0 -> 14
Other:
- note added: "+5V Regulator"
- note added: "3.3V/1.8V regulators"
- note added: "Backlight Circuitry"
- note added: "Battery Holder"
- note added: "Decoupling"
- note added: "LED Current Sink Driver"
- note added: "RX5808 Circuitry"
- note added: "Status LEDs"
- note added: "TFT Display"
- note added: "TFT Display Conn"
- note added: "TW8819 Circuitry"
- note added: "USB C and Bat Charger"
- note added: "Voltage Booster for Backlight"

Commit message: Update
Parts:
- C100: value 33uF -> 10uF
- C101: value 10uF -> 1uF
- C98: footprint Capacitor_SMD:C_0603_1608Metric -> Capacitor_SMD:C_1206_3216Metric
- C99: value 4.7uF -> 1uF
Changed lines of the file:
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@@
 			)
 		)
-		(property "Value" "10uF"
+		(property "Value" "1uF"
 			(at 117.602 50.8 0)
 			(effects
@@
 			)
 		)
-		(property "Value" "33uF"
+		(property "Value" "10uF"
 			(at 72.644 52.578 0)
 			(effects
@@
 			)
 		)
-		(property "Value" "4.7uF"
+		(property "Value" "1uF"
 			(at 69.342 40.64 0)
 			(effects
@@
 			)
 		)
-		(property "Footprint" "Capacitor_SMD:C_0603_1608Metric"
+		(property "Footprint" "Capacitor_SMD:C_1206_3216Metric"
 			(at 206.0448 181.61 0)
 			(effects
